File: MCU.kicad_sch (KiCad schematic)
At the start: 0 parts

Commit message: added micro and 3 sensors and connectors with USB
Parts:
- added C1, C2, C24, C3, C4, C5: 100nF, Capacitor_SMD:C_0603_1608Metric, symbol Device:C
- added C20: 4.7uF 10V, Capacitor_SMD:C_0603_1608Metric, symbol Device:C
- added C21, C22: 2.2uF 10V, Capacitor_SMD:C_0603_1608Metric, symbol Device:C
- added C23: 1uF 10V, Capacitor_SMD:C_0603_1608Metric, symbol Device:C
- added C25, C26: 12pF C0G, Capacitor_SMD:C_0603_1608Metric, symbol Device:C
- added FB1: 600R@100MHz, Inductor_SMD:L_0603_1608Metric, symbol Device:FerriteBead
- added R1: 10k, Resistor_SMD:R_0603_1608Metric, symbol Device:R
- added SW1: BOOT0, Button_Switch_SMD:SW_SPST_TL3342, symbol Switch:SW_Push
- added U1: STM32F405RGTx, Package_QFP:LQFP-64_10x10mm_P0.5mm, symbol MCU_ST_STM32F4:STM32F405RGTx
- added Y1: 8MHz, Crystal:Crystal_SMD_Abracon_ABM3B-4Pin_5.0x3.2mm, symbol Device:Crystal_GND24
Connections:
- new net: C23.1, C24.1, FB1.2, U1.13 (VDDA)
- new net: C21.1, U1.31 (VCAP_1)
- new net: C22.1, U1.47 (VCAP_2)
- new net: R1.1, SW1.2, U1.60 (BOOT0)
- new net 3V3: C1.1, C2.1, C20.1, C3.1, C4.1, FB1.1, SW1.1, U1.1 (VBAT), U1.19 (VDD), U1.32 (VDD), U1.48 (VDD), U1.64 (VDD)
- new net ACC_INT1: U1.27 (PB1)
- new net CAM_RX: U1.38 (PC7)
- new net CAM_TX: U1.37 (PC6)
- new net CS_ACC: U1.24 (PC4)
- new net CS_BAR: U1.25 (PC5)
- new net CS_IMU: U1.20 (PA4)
- new net DBG_RX: U1.30 (PB11)
- new net DBG_TX: U1.29 (PB10)
- new net GND: C1.2, C2.2, C20.2, C21.2, C22.2, C23.2, C24.2, C25.2, C26.2, C3.2, C4.2, C5.2, R1.2, U1.12 (VSSA), U1.18 (VSS), U1.63 (VSS), Y1.2 (G), Y1.4 (G)
- new net IMU_INT1: U1.26 (PB0)
- new net NRST: C5.1, U1.7 (NRST)
- new net OSC_IN: C25.1, U1.5 (PH0), Y1.1
- new net OSC_OUT: C26.1, U1.6 (PH1), Y1.3
- new net SCL: U1.21 (PA5)
- new net SDA: U1.23 (PA7)
- new net SDO: U1.22 (PA6)
- new net SWCLK: U1.49 (PA14)
- new net SWDIO: U1.46 (PA13)
- new net SWO: U1.55 (PB3)
- new net USB_DM: U1.44 (PA11)
- new net USB_DP: U1.45 (PA12)

Commit message: added GPS and Temp/Humid sensor
Connections:
- net TIMER_GPS: now reaches U1.14 (PA0)
- net RX_GPS: now reaches U1.16 (PA2)
- net TX_GPS: now reaches U1.17 (PA3)
- net RESET_GPS: now reaches U1.56 (PB4)
- net SCL_T: now reaches U1.58 (PB6)
- net SDA_T: now reaches U1.59 (PB7)
Other:
- moved on the sheet: C1, C2, C20, C21, C22, C23, C24, C25, C26, C3, C4, C5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

Commit message: added Buzzer, status LEDs
Parts:
- added BZ1: CMT-8504-100-SMT, Buzzer_Beeper:MagneticBuzzer_CUI_CMT-8504-100-SMT, symbol Device:Buzzer
- added C33: 100nF, Capacitor_SMD:C_0603_1608Metric, symbol Device:C
- added D2: Green, LED_SMD:LED_0603_1608Metric, symbol Device:LED
- added D3: B5819W, Diode_SMD:D_SOD-123, symbol Device:D_Schottky
- added Q2: AO3400A, Package_TO_SOT_SMD:SOT-23, symbol Transistor_FET:AO3400A
- added R16: 100k 1%, Resistor_SMD:R_0603_1608Metric, symbol Device:R
- added R17: 33k 1%, Resistor_SMD:R_0603_1608Metric, symbol Device:R
- added R18: 10k, Resistor_SMD:R_0603_1608Metric, symbol Device:R
- added R19: 330R, Resistor_SMD:R_0603_1608Metric, symbol Device:R
- added R20: 100R, Resistor_SMD:R_0603_1608Metric, symbol Device:R
- added R21: 100k, Resistor_SMD:R_0603_1608Metric, symbol Device:R
Connections:
- net GND: now also C33.2, D2.1 (K), Q2.2 (S), R17.2, R18.2, R21.2
- net at U1.10 (PC2): now also R19.2
- net VBAT_SENSE: now reaches U1.15 (PA1)
- net VBAT_SENSE: now also C33.1, R16.2, R17.1
- net BOOT1: now reaches U1.28 (PB2)
- net BOOT1: now also R18.1
- net LORA_CS: now reaches U1.33 (PB12)
- net LORA_SCK: now reaches U1.34 (PB13)
- net LORA_MISO: now reaches U1.35 (PB14)
- net LORA_MOSI: now reaches U1.36 (PB15)
- net LORA_BUSY: now reaches U1.39 (PC8)
- net LORA_DIO1: now reaches U1.40 (PC9)
- net LORA_NRST: now reaches U1.41 (PA8)
- net CS_FLASH: now reaches U1.50 (PA15)
- net CLK_FLASH: now reaches U1.51 (PC10)
- net DO_FLASH: now reaches U1.52 (PC11)
- net DI_FLASH: now reaches U1.53 (PC12)
- net LORA_RXEN: now reaches U1.57 (PB5)
- net BUZZER: now reaches U1.61 (PB8)
- net BUZZER: now also R20.1, R21.1
- new net: BZ1.2 (-), D3.2 (A), Q2.3 (D)
- new net: D2.2 (A), R19.1
- new net: Q2.1 (G), R20.2
- new net +BATT: R16.1
- new net 5V0: BZ1.1 (+), D3.1 (K)

Commit message: Battery protection, camera switch, 64MB flash, ERC clean
- Fuse + TVS on battery input, camera load switch (TPS22917)
- Flash to W25Q512JVFIQ (SOIC-16), hand-solder passive footprints
- Power LED, title blocks, U5 footprint, PWR/NC flags (0 ERC)
- Regenerated schematic PDF
Parts:
- C1, C2, C20, C21, C22, C23, C24, C25, C26, C3, C33, C4, C5: footprint Capacitor_SMD:C_0603_1608Metric -> Capacitor_SMD:C_0603_1608Metric_Pad1.08x0.95mm_HandSolder
- D2: footprint LED_SMD:LED_0603_1608Metric -> LED_SMD:LED_0603_1608Metric_Pad1.05x0.95mm_HandSolder
- FB1: footprint Inductor_SMD:L_0603_1608Metric -> Inductor_SMD:L_0603_1608Metric_Pad1.05x0.95mm_HandSolder
- R1, R16, R17, R18, R19, R20, R21: footprint Resistor_SMD:R_0603_1608Metric -> Resistor_SMD:R_0603_1608Metric_Pad0.98x0.95mm_HandSolder
Connections:
- net CAM_EN: now reaches U1.2 (PC13)
- no-connect marks 0 -> 9
Other:
- title: (none) -> Microcontroller: STM32F405
- moved on the sheet: C33, D3, R21
